File: BACEE.sch (KiCad schematic (older format))
At the start: 13 parts

Commit message: Annotated and edited symbol values.
Parts:
- BT1: renamed from BT?; value Battery -> Battery 3V; footprint (none) -> Connector_PinHeader_2.54mm:PinHeader_1x02_P2.54mm_Vertical
- C1, C2: renamed from C?; value C -> 22pF; footprint (none) -> Capacitor_SMD:C_0805_2012Metric_Pad1.15x1.40mm_HandSolder
- C3: renamed from C?; value CP1 -> 10uF; footprint (none) -> Capacitor_SMD:C_0805_2012Metric_Pad1.15x1.40mm_HandSolder
- D1: renamed from D?; footprint (none) -> LED_SMD:LED_0805_2012Metric_Pad1.15x1.40mm_HandSolder
- R1: renamed from R?; value R -> 330Ohm; footprint (none) -> Resistor_SMD:R_0805_2012Metric_Pad1.15x1.40mm_HandSolder
- R2: renamed from R?; value R -> 10kOhm; footprint (none) -> Resistor_SMD:R_0805_2012Metric_Pad1.15x1.40mm_HandSolder
- U1, U3: renamed from U?; footprint (none) -> Package_SO:SOIJ-8_5.3x5.3mm_P1.27mm
- U2: renamed from U?; footprint (none) -> Package_SO:SO-8_5.3x6.2mm_P1.27mm
- Y1: renamed from Y?; value Crystal -> Crystal32768KHz; footprint (none) -> Crystal:Crystal_SMD_MicroCrystal_CC7V-T1A-2Pin_3.2x1.5mm_HandSoldering
- Y2: renamed from Y?; value Crystal -> Crystal 16MHz; footprint (none) -> Crystal:Crystal_SMD_5032-2Pin_5.0x3.2mm_HandSoldering
- gave numbers to parts that had none: 1
Changed lines of the file:
@@
 $EndDescr
 $Comp
-L Peters_library:DS1337S+ U?
+L Peters_library:DS1337S+ U2
 U 1 1 5B7FD1F4
 P 2900 1900
-F 0 "U?" H 2900 2528 50  0000 C CNN
+F 0 "U2" H 2900 2528 50  0000 C CNN
 F 1 "DS1337S+" H 2900 2437 50  0000 C CNN
-F 2 "" H 2900 2000 50  0001 C CNN
+F 2 "Package_SO:SO-8_5.3x6.2mm_P1.27mm" H 2900 2000 50  0001 C CNN
 F 3 "" H 2900 2000 50  0001 C CNN
 	1    2900 1900
@@
 $EndComp
 $Comp
-L Memory_EEPROM:24LC1025 U?
+L Memory_EEPROM:24LC1025 U1
 U 1 1 5B7FD31C
 P 2400 4150
-F 0 "U?" H 2400 4628 50  0000 C CNN
+F 0 "U1" H 2400 4628 50  0000 C CNN
 F 1 "24LC1025" H 2400 4537 50  0000 C CNN
-F 2 "" H 2400 4150 50  0001 C CNN
+F 2 "Package_SO:SOIJ-8_5.3x5.3mm_P1.27mm" H 2400 4150 50  0001 C CNN
 F 3 "http://ww1.microchip.com/downloads/en/DeviceDoc/21941B.pdf" H 2400 4150 50  0001 C CNN
 	1    2400 4150
@@
 $EndComp
 $Comp
-L Memory_EEPROM:24LC1025 U?
+L Memory_EEPROM:24LC1025 U3
 U 1 1 5B7FD368
 P 3900 4150
-F 0 "U?" H 3900 4628 50  0000 C CNN
+F 0 "U3" H 3900 4628 50  0000 C CNN
 F 1 "24LC1025" H 3900 4537 50  0000 C CNN
-F 2 "" H 3900 4150 50  0001 C CNN
+F 2 "Package_SO:SOIJ-8_5.3x5.3mm_P1.27mm" H 3900 4150 50  0001 C CNN
 F 3 "http://ww1.microchip.com/downloads/en/DeviceDoc/21941B.pdf" H 3900 4150 50  0001 C CNN
 	1    3900 4150
@@
 $EndComp
 $Comp
-L dk_Embedded-Microcontrollers:ATMEGA328P-AU U?
+L dk_Embedded-Microcontrollers:ATMEGA328P-AU U4
 U 1 1 5B7FD68A
 P 7600 3200
-F 0 "U?" H 7928 3303 60  0000 L CNN
+F 0 "U4" H 7928 3303 60  0000 L CNN
 F 1 "ATMEGA328P-AU" H 7928 3197 60  0000 L CNN
 F 2 "digikey-footprints:TQFP-32_7x7mm" H 7800 3400 60  0001 L CNN
@@
 $EndComp
 $Comp
-L Device:C C?
+L Device:C C1
 U 1 1 5B7FD778
 P 5750 1700
-F 0 "C?" V 5498 1700 50  0000 C CNN
-F 1 "C" V 5589 1700 50  0000 C CNN
-F 2 "" H 5788 1550 50  0001 C CNN
+F 0 "C1" V 5498 1700 50  0000 C CNN
+F 1 "22pF" V 5589 1700 50  0000 C CNN
+F 2 "Capacitor_SMD:C_0805_2012Metric_Pad1.15x1.40mm_HandSolder" H 5788 1550 50  0001 C CNN
 F 3 "~" H 5750 1700 50  0001 C CNN
 	1    5750 1700
@@
 $EndComp
 $Comp
-L Device:C C?
+L Device:C C2
 U 1 1 5B7FD7CA
 P 5750 2350
-F 0 "C?" V 5498 2350 50  0000 C CNN
-F 1 "C" V 5589 2350 50  0000 C CNN
-F 2 "" H 5788 2200 50  0001 C CNN
+F 0 "C2" V 5498 2350 50  0000 C CNN
+F 1 "22pF" V 5589 2350 50  0000 C CNN
+F 2 "Capacitor_SMD:C_0805_2012Metric_Pad1.15x1.40mm_HandSolder" H 5788 2200 50  0001 C CNN
 F 3 "~" H 5750 2350 50  0001 C CNN
 	1    5750 2350
@@
 $EndComp
 $Comp
-L Device:CP1 C?
+L Device:CP1 C3
 U 1 1 5B7FD83B
 P 9350 2550
-F 0 "C?" H 9465 2596 50  0000 L CNN
-F 1 "CP1" H 9465 2505 50  0000 L CNN
-F 2 "" H 9350 2550 50  0001 C CNN
+F 0 "C3" H 9465 2596 50  0000 L CNN
+F 1 "10uF" H 9465 2505 50  0000 L CNN
+F 2 "Capacitor_SMD:C_0805_2012Metric_Pad1.15x1.40mm_HandSolder" H 9350 2550 50  0001 C CNN
 F 3 "~" H 9350 2550 50  0001 C CNN
 	1    9350 2550
@@
 $EndComp
 $Comp
-L Device:R R?
+L Device:R R1
 U 1 1 5B7FD90B
 P 5900 3250
-F 0 "R?" H 5970 3296 50  0000 L CNN
-F 1 "R" H 5970 3205 50  0000 L CNN
-F 2 "" V 5830 3250 50  0001 C CNN
+F 0 "R1" H 5830 3204 50  0000 R CNN
+F 1 "330Ohm" H 5830 3295 50  0000 R CNN
+F 2 "Resistor_SMD:R_0805_2012Metric_Pad1.15x1.40mm_HandSolder" V 5830 3250 50  0001 C CNN
 F 3 "~" H 5900 3250 50  0001 C CNN
 	1    5900 3250
-	1    0    0    -1
+	-1   0    0    1
 $EndComp
 $Comp
-L Device:R R?
+L Device:R R2
 U 1 1 5B7FD977
 P 6350 4050
-F 0 "R?" H 6420 4096 50  0000 L CNN
-F 1 "R" H 6420 4005 50  0000 L CNN
-F 2 "" V 6280 4050 50  0001 C CNN
+F 0 "R2" H 6420 4096 50  0000 L CNN
+F 1 "10kOhm" H 6420 4005 50  0000 L CNN
+F 2 "Resistor_SMD:R_0805_2012Metric_Pad1.15x1.40mm_HandSolder" V 6280 4050 50  0001 C CNN
 F 3 "~" H 6350 4050 50  0001 C CNN
 	1    6350 4050
@@
 $EndComp
 $Comp
-L Device:LED D?
+L Device:LED D1
 U 1 1 5B7FDA0F
 P 6300 2850
-F 0 "D?" H 6291 3066 50  0000 C CNN
+F 0 "D1" H 6291 3066 50  0000 C CNN
 F 1 "LED" H 6291 2975 50  0000 C CNN
-F 2 "" H 6300 2850 50  0001 C CNN
+F 2 "LED_SMD:LED_0805_2012Metric_Pad1.15x1.40mm_HandSolder" H 6300 2850 50  0001 C CNN
 F 3 "~" H 6300 2850 50  0001 C CNN
 	1    6300 2850
@@
 $EndComp
 $Comp
-L Device:Crystal Y?
+L Device:Crystal Y1
 U 1 1 5B7FDADF
-P 1650 1800
-F 0 "Y?" V 1604 1931 50  0000 L CNN
-F 1 "Crystal" V 1695 1931 50  0000 L CNN
-F 2 "" H 1650 1800 50  0001 C CNN
-F 3 "~" H 1650 1800 50  0001 C CNN
-	1    1650 1800
-	0    1    1    0
+P 1500 1800
+F 0 "Y1" V 1546 1669 50  0000 R CNN
+F 1 "Crystal32768KHz" V 1455 1669 50  0000 R CNN
+F 2 "Crystal:Crystal_SMD_MicroCrystal_CC7V-T1A-2Pin_3.2x1.5mm_HandSoldering" H 1500 1800 50  0001 C CNN
+F 3 "~" H 1500 1800 50  0001 C CNN
+	1    1500 1800
+	0    -1   -1   0
 $EndComp
 $Comp
-L Device:Crystal Y?
+L Device:Crystal Y2
 U 1 1 5B7FDB6F
 P 6300 2000
-F 0 "Y?" V 6254 2131 50  0000 L CNN
-F 1 "Crystal" V 6345 2131 50  0000 L CNN
-F 2 "" H 6300 2000 50  0001 C CNN
+F 0 "Y2" V 6254 2131 50  0000 L CNN
+F 1 "Crystal 16MHz" V 6345 2131 50  0000 L CNN
+F 2 "Crystal:Crystal_SMD_5032-2Pin_5.0x3.2mm_HandSoldering" H 6300 2000 50  0001 C CNN
 F 3 "~" H 6300 2000 50  0001 C CNN
 	1    6300 2000
@@
 $EndComp
 $Comp
-L Device:Battery BT?
+L Device:Battery BT1
 U 1 1 5B7FDC29
 P 9900 2550
-F 0 "BT?" H 10008 2596 50  0000 L CNN
-F 1 "Battery" H 10008 2505 50  0000 L CNN
-F 2 "" V 9900 2610 50  0001 C CNN
+F 0 "BT1" H 10008 2596 50  0000 L CNN
+F 1 "Battery 3V" H 10008 2505 50  0000 L CNN
+F 2 "Connector_PinHeader_2.54mm:PinHeader_1x02_P2.54mm_Vertical" V 9900 2610 50  0001 C CNN
 F 3 "~" V 9900 2610 50  0001 C CNN
 	1    9900 2550
@@
 $EndComp
 $Comp
-L power:GND #PWR?
+L power:GND #PWR02
 U 1 1 5B7FDCEB
 P 9900 3150
-F 0 "#PWR?" H 9900 2900 50  0001 C CNN
+F 0 "#PWR02" H 9900 2900 50  0001 C CNN
 F 1 "GND" H 9905 2977 50  0000 C CNN
 F 2 "" H 9900 3150 50  0001 C CNN
@@
 $EndSheet
 $Comp
-L power:GND #PWR?
+L power:GND #PWR01
 U 1 1 5B7FEA2F
 P 1850 6400
-F 0 "#PWR?" H 1850 6150 50  0001 C CNN
+F 0 "#PWR01" H 1850 6150 50  0001 C CNN
 F 1 "GND" H 1855 6227 50  0000 C CNN
 F 2 "" H 1850 6400 50  0001 C CNN

Commit message: Wired MCU.
Connections:
- net labels added: ADDS1, ADDS2, D2, D3, D4, D5, D6, D7, D8, MISO, MOSI, RESET, RX, TX
- wire segments 5 -> 56
- no-connect marks 0 -> 7

Commit message: Wired main symbols.
Connections:
- wire segments 56 -> 67
- no-connect marks 7 -> 8
Changed lines of the file:
@@
 U 1 1 5B7FD1F4
 P 2900 1900
-F 0 "U2" H 2900 2528 50  0000 C CNN
-F 1 "DS1337S+" H 2900 2437 50  0000 C CNN
+F 0 "U2" H 3250 2350 50  0000 C CNN
+F 1 "DS1337S+" H 2500 2350 50  0000 C CNN
 F 2 "Package_SO:SO-8_5.3x6.2mm_P1.27mm" H 2900 2000 50  0001 C CNN
 F 3 "" H 2900 2000 50  0001 C CNN
@@
 U 1 1 5B7FD31C
 P 2400 4150
-F 0 "U1" H 2400 4628 50  0000 C CNN
-F 1 "24LC1025" H 2400 4537 50  0000 C CNN
+F 0 "U1" H 2650 4450 50  0000 C CNN
+F 1 "24LC1025" H 2050 4450 50  0000 C CNN
 F 2 "Package_SO:SOIJ-8_5.3x5.3mm_P1.27mm" H 2400 4150 50  0001 C CNN
 F 3 "http://ww1.microchip.com/downloads/en/DeviceDoc/21941B.pdf" H 2400 4150 50  0001 C CNN
@@
 U 1 1 5B7FD368
 P 3900 4150
-F 0 "U3" H 3900 4628 50  0000 C CNN
-F 1 "24LC1025" H 3900 4537 50  0000 C CNN
+F 0 "U3" H 4150 4450 50  0000 C CNN
+F 1 "24LC1025" H 3550 4450 50  0000 C CNN
 F 2 "Package_SO:SOIJ-8_5.3x5.3mm_P1.27mm" H 3900 4150 50  0001 C CNN
 F 3 "http://ww1.microchip.com/downloads/en/DeviceDoc/21941B.pdf" H 3900 4150 50  0001 C CNN
@@
 Vcc
 Wire Wire Line
-	9450 1350 7800 1350
+	9450 1350 8850 1350
 Connection ~ 7800 1350
 Wire Wire Line
@@
 Wire Wire Line
 	7700 4800 7700 4850
+NoConn ~ 3350 1700
+Text Label 3350 1900 0    50   ~ 0
+SCK
+Text Label 2800 4150 0    50   ~ 0
+SCK
+Text Label 4300 4150 0    50   ~ 0
+SCK
+Text Label 3350 2100 0    50   ~ 0
+SDA
+Text Label 2800 4050 0    50   ~ 0
+SDA
+Text Label 4300 4050 0    50   ~ 0
+SDA
+Text Label 2000 4050 2    50   ~ 0
+ADDS1
+Text Label 3500 4050 2    50   ~ 0
+ADDS1
+Text Label 2000 4150 2    50   ~ 0
+ADDS2
+Text Label 3500 4150 2    50   ~ 0
+ADDS2
+$Comp
+L power:GND #PWR?
+U 1 1 5B8142A1
+P 2900 2600
+F 0 "#PWR?" H 2900 2350 50  0001 C CNN
+F 1 "GND" H 2905 2427 50  0000 C CNN
+F 2 "" H 2900 2600 50  0001 C CNN
+F 3 "" H 2900 2600 50  0001 C CNN
+	1    2900 2600
+	1    0    0    -1
+$EndComp
+Wire Wire Line
+	2900 2350 2900 2600
+Text Label 2900 1300 0    50   ~ 0
+Vcc
+Wire Wire Line
+	2900 1450 2900 1300
+Text Label 2450 2100 2    50   ~ 0
+Vcc
+Text Label 2000 4250 2    50   ~ 0
+Vcc
+Text Label 3500 4250 2    50   ~ 0
+Vcc
+Text Label 2400 3650 2    50   ~ 0
+Vcc
+Wire Wire Line
+	2400 3850 2400 3650
+Wire Wire Line
+	3900 3850 3900 3650
+Text Label 3900 3650 2    50   ~ 0
+Vcc
+Wire Wire Line
+	2400 4450 2400 4600
+Wire Wire Line
+	2400 4600 3150 4600
+Wire Wire Line
+	3900 4600 3900 4450
+$Comp
+L power:GND #PWR?
+U 1 1 5B81A59B
+P 3150 4700
+F 0 "#PWR?" H 3150 4450 50  0001 C CNN
+F 1 "GND" H 3155 4527 50  0000 C CNN
+F 2 "" H 3150 4700 50  0001 C CNN
+F 3 "" H 3150 4700 50  0001 C CNN
+	1    3150 4700
+	1    0    0    -1
+$EndComp
+Wire Wire Line
+	3150 4700 3150 4600
+Connection ~ 3150 4600
+Wire Wire Line
+	3150 4600 3900 4600
+$Comp
+L power:PWR_FLAG #FLG?
+U 1 1 5B81BD18
+P 8850 1200
+F 0 "#FLG?" H 8850 1275 50  0001 C CNN
+F 1 "PWR_FLAG" H 8850 1374 50  0000 C CNN
+F 2 "" H 8850 1200 50  0001 C CNN
+F 3 "~" H 8850 1200 50  0001 C CNN
+	1    8850 1200
+	1    0    0    -1
+$EndComp
+Wire Wire Line
+	8850 1200 8850 1350
+Connection ~ 8850 1350
+Wire Wire Line
+	8850 1350 7800 1350
 $EndSCHEMATC

Commit message: Labeled sheet rectangle.
Connections:
- wire segments 67 -> 79
Other:
- moved on the sheet: U1, U3
Changed lines of the file:
@@
 L Peters_library:DS1337S+ U2
 U 1 1 5B7FD1F4
-P 2900 1900
-F 0 "U2" H 3250 2350 50  0000 C CNN
-F 1 "DS1337S+" H 2500 2350 50  0000 C CNN
-F 2 "Package_SO:SO-8_5.3x6.2mm_P1.27mm" H 2900 2000 50  0001 C CNN
-F 3 "" H 2900 2000 50  0001 C CNN
-	1    2900 1900
+P 3650 1750
+F 0 "U2" H 4000 2200 50  0000 C CNN
+F 1 "DS1337S+" H 3250 2200 50  0000 C CNN
+F 2 "Package_SO:SO-8_5.3x6.2mm_P1.27mm" H 3650 1850 50  0001 C CNN
+F 3 "" H 3650 1850 50  0001 C CNN
+	1    3650 1750
 	1    0    0    -1
 $EndComp
@@
 L Memory_EEPROM:24LC1025 U1
 U 1 1 5B7FD31C
-P 2400 4150
-F 0 "U1" H 2650 4450 50  0000 C CNN
-F 1 "24LC1025" H 2050 4450 50  0000 C CNN
-F 2 "Package_SO:SOIJ-8_5.3x5.3mm_P1.27mm" H 2400 4150 50  0001 C CNN
-F 3 "http://ww1.microchip.com/downloads/en/DeviceDoc/21941B.pdf" H 2400 4150 50  0001 C CNN
-	1    2400 4150
+P 3150 4000
+F 0 "U1" H 3400 4300 50  0000 C CNN
+F 1 "24LC1025" H 2800 4300 50  0000 C CNN
+F 2 "Package_SO:SOIJ-8_5.3x5.3mm_P1.27mm" H 3150 4000 50  0001 C CNN
+F 3 "http://ww1.microchip.com/downloads/en/DeviceDoc/21941B.pdf" H 3150 4000 50  0001 C CNN
+	1    3150 4000
 	1    0    0    -1
 $EndComp
@@
 L Memory_EEPROM:24LC1025 U3
 U 1 1 5B7FD368
-P 3900 4150
-F 0 "U3" H 4150 4450 50  0000 C CNN
-F 1 "24LC1025" H 3550 4450 50  0000 C CNN
-F 2 "Package_SO:SOIJ-8_5.3x5.3mm_P1.27mm" H 3900 4150 50  0001 C CNN
-F 3 "http://ww1.microchip.com/downloads/en/DeviceDoc/21941B.pdf" H 3900 4150 50  0001 C CNN
-	1    3900 4150
+P 4650 4000
+F 0 "U3" H 4900 4300 50  0000 C CNN
+F 1 "24LC1025" H 4300 4300 50  0000 C CNN
+F 2 "Package_SO:SOIJ-8_5.3x5.3mm_P1.27mm" H 4650 4000 50  0001 C CNN
+F 3 "http://ww1.microchip.com/downloads/en/DeviceDoc/21941B.pdf" H 4650 4000 50  0001 C CNN
+	1    4650 4000
 	1    0    0    -1
 $EndComp
@@
 L Device:Crystal Y1
 U 1 1 5B7FDADF
-P 1500 1800
-F 0 "Y1" V 1546 1669 50  0000 R CNN
-F 1 "Crystal32768KHz" V 1455 1669 50  0000 R CNN
-F 2 "Crystal:Crystal_SMD_MicroCrystal_CC7V-T1A-2Pin_3.2x1.5mm_HandSoldering" H 1500 1800 50  0001 C CNN
-F 3 "~" H 1500 1800 50  0001 C CNN
-	1    1500 1800
+P 2250 1650
+F 0 "Y1" V 2296 1519 50  0000 R CNN
+F 1 "Crystal32768KHz" V 2205 1519 50  0000 R CNN
+F 2 "Crystal:Crystal_SMD_MicroCrystal_CC7V-T1A-2Pin_3.2x1.5mm_HandSoldering" H 2250 1650 50  0001 C CNN
+F 3 "~" H 2250 1650 50  0001 C CNN
+	1    2250 1650
 	0    -1   -1   0
 $EndComp
@@
 F0 "Connectors" 50
 F1 "Connectors.sch" 50
-F2 "GND" I L 2450 6300 50
-F3 "Vcc" I L 2450 6450 50
-F4 "SDA" B L 2450 6600 50
-F5 "SCK" B L 2450 6750 50
+F2 "GND" I L 2450 6200 50
+F3 "Vcc" I L 2450 6300 50
+F4 "SDA" B L 2450 6400 50
+F5 "SCK" B L 2450 6500 50
+F6 "MISO" O L 2450 7100 50
+F7 "RESET" O L 2450 6900 50
+F8 "MOSI" I L 2450 7000 50
+F9 "D2" B R 3400 6200 50
+F10 "D3" B R 3400 6300 50
+F11 "D4" B R 3400 6400 50
+F12 "D5" B R 3400 6500 50
+F13 "D6" B R 3400 6600 50
+F14 "D7" B R 3400 6700 50
+F15 "D8" B R 3400 6800 50
+F16 "RX" I L 2450 6750 50
+F17 "TX" O L 2450 6650 50
 $EndSheet
 $Comp
@@
 	1    0    0    -1
 $EndComp
-Wire Wire Line
-	1850 6400 1850 6300
-Wire Wire Line
-	1850 6300 2450 6300
-Wire Wire Line
-	2450 6450 2200 6450
-Wire Wire Line
-	2450 6600 2200 6600
-Wire Wire Line
-	2450 6750 2200 6750
-Text Label 2200 6450 2    50   ~ 0
-Vcc
-Text Label 2200 6600 2    50   ~ 0
+Text Label 2350 6300 2    50   ~ 0
+Vcc
+Text Label 2350 6400 2    50   ~ 0
 SDA
-Text Label 2200 6750 2    50   ~ 0
+Text Label 2350 6500 2    50   ~ 0
 SCK
 Wire Wire Line
@@
 Connection ~ 7800 1350
 Wire Wire Line
-	2450 1700 2100 1700
-Wire Wire Line
-	2100 1700 2100 1550
-Wire Wire Line
-	2100 1550 1500 1550
-Wire Wire Line
-	1500 1550 1500 1650
-Wire Wire Line
-	2450 1900 2100 1900
-Wire Wire Line
-	2100 1900 2100 2100
-Wire Wire Line
-	2100 2100 1500 2100
-Wire Wire Line
-	1500 2100 1500 1950
+	3200 1550 2850 1550
+Wire Wire Line
+	2850 1550 2850 1400
+Wire Wire Line
+	2850 1400 2250 1400
+Wire Wire Line
+	2250 1400 2250 1500
+Wire Wire Line
+	3200 1750 2850 1750
+Wire Wire Line
+	2850 1750 2850 1950
+Wire Wire Line
+	2850 1950 2250 1950
+Wire Wire Line
+	2250 1950 2250 1800
 Text Label 7100 1900 2    50   ~ 0
 D3
@@
 Wire Wire Line
 	7700 4800 7700 4850
-NoConn ~ 3350 1700
-Text Label 3350 1900 0    50   ~ 0
+NoConn ~ 4100 1550
+Text Label 4100 1750 0    50   ~ 0
 SCK
-Text Label 2800 4150 0    50   ~ 0
+Text Label 3550 4000 0    50   ~ 0
 SCK
-Text Label 4300 4150 0    50   ~ 0
+Text Label 5050 4000 0    50   ~ 0
 SCK
-Text Label 3350 2100 0    50   ~ 0
+Text Label 4100 1950 0    50   ~ 0
 SDA
-Text Label 2800 4050 0    50   ~ 0
+Text Label 3550 3900 0    50   ~ 0
 SDA
-Text Label 4300 4050 0    50   ~ 0
+Text Label 5050 3900 0    50   ~ 0
 SDA
-Text Label 2000 4050 2    50   ~ 0
+Text Label 2750 3900 2    50   ~ 0
 ADDS1
-Text Label 3500 4050 2    50   ~ 0
+Text Label 4250 3900 2    50   ~ 0
 ADDS1
-Text Label 2000 4150 2    50   ~ 0
+Text Label 2750 4000 2    50   ~ 0
 ADDS2
-Text Label 3500 4150 2    50   ~ 0
+Text Label 4250 4000 2    50   ~ 0
 ADDS2
 $Comp
 L power:GND #PWR?
 U 1 1 5B8142A1
-P 2900 2600
-F 0 "#PWR?" H 2900 2350 50  0001 C CNN
-F 1 "GND" H 2905 2427 50  0000 C CNN
-F 2 "" H 2900 2600 50  0001 C CNN
-F 3 "" H 2900 2600 50  0001 C CNN
-	1    2900 2600
-	1    0    0    -1
-$EndComp
-Wire Wire Line
-	2900 2350 2900 2600
-Text Label 2900 1300 0    50   ~ 0
-Vcc
-Wire Wire Line
-	2900 1450 2900 1300
-Text Label 2450 2100 2    50   ~ 0
-Vcc
-Text Label 2000 4250 2    50   ~ 0
-Vcc
-Text Label 3500 4250 2    50   ~ 0
-Vcc
-Text Label 2400 3650 2    50   ~ 0
-Vcc
-Wire Wire Line
-	2400 3850 2400 3650
-Wire Wire Line
-	3900 3850 3900 3650
-Text Label 3900 3650 2    50   ~ 0
-Vcc
-Wire Wire Line
-	2400 4450 2400 4600
-Wire Wire Line
-	2400 4600 3150 4600
-Wire Wire Line
-	3900 4600 3900 4450
+P 3650 2450
+F 0 "#PWR?" H 3650 2200 50  0001 C CNN
+F 1 "GND" H 3655 2277 50  0000 C CNN
+F 2 "" H 3650 2450 50  0001 C CNN
+F 3 "" H 3650 2450 50  0001 C CNN
+	1    3650 2450
+	1    0    0    -1
+$EndComp
+Wire Wire Line
+	3650 2200 3650 2450
+Text Label 3650 1150 0    50   ~ 0
+Vcc
+Wire Wire Line
+	3650 1300 3650 1150
+Text Label 3200 1950 2    50   ~ 0
+Vcc
+Text Label 2750 4100 2    50   ~ 0
+Vcc
+Text Label 4250 4100 2    50   ~ 0
+Vcc
+Text Label 3150 3500 2    50   ~ 0
+Vcc
+Wire Wire Line
+	3150 3700 3150 3500
+Wire Wire Line
+	4650 3700 4650 3500
+Text Label 4650 3500 2    50   ~ 0
+Vcc
+Wire Wire Line
+	3150 4300 3150 4450
+Wire Wire Line
+	3150 4450 3900 4450
+Wire Wire Line
+	4650 4450 4650 4300
 $Comp
 L power:GND #PWR?
 U 1 1 5B81A59B
-P 3150 4700
-F 0 "#PWR?" H 3150 4450 50  0001 C CNN
-F 1 "GND" H 3155 4527 50  0000 C CNN
-F 2 "" H 3150 4700 50  0001 C CNN
-F 3 "" H 3150 4700 50  0001 C CNN
-	1    3150 4700
-	1    0    0    -1
-$EndComp
-Wire Wire Line
-	3150 4700 3150 4600
-Connection ~ 3150 4600
-Wire Wire Line
-	3150 4600 3900 4600
+P 3900 4550
+F 0 "#PWR?" H 3900 4300 50  0001 C CNN
+F 1 "GND" H 3905 4377 50  0000 C CNN
+F 2 "" H 3900 4550 50  0001 C CNN
+F 3 "" H 3900 4550 50  0001 C CNN
+	1    3900 4550
+	1    0    0    -1
+$EndComp
+Wire Wire Line
+	3900 4550 3900 4450
+Connection ~ 3900 4450
+Wire Wire Line
+	3900 4450 4650 4450
 $Comp
 L power:PWR_FLAG #FLG?
@@
 Wire Wire Line
 	8850 1350 7800 1350
+Wire Wire Line
+	1850 6200 2450 6200
+Wire Wire Line
+	1850 6200 1850 6400
+Wire Wire Line
+	2450 6300 2350 6300
+Wire Wire Line
+	2450 6400 2350 6400
+Wire Wire Line
+	2450 6500 2350 6500
+Wire Wire Line
+	2450 6650 2350 6650
+Wire Wire Line
+	2450 6750 2350 6750
+Wire Wire Line
+	2450 6900 2350 6900
+Wire Wire Line
+	2450 7000 2350 7000
+Wire Wire Line
+	2450 7100 2350 7100
+Wire Wire Line
+	3400 6200 3500 6200
+Wire Wire Line
+	3400 6300 3500 6300
+Wire Wire Line
+	3400 6400 3500 6400
+Wire Wire Line
+	3400 6500 3500 6500
+Wire Wire Line
+	3400 6600 3500 6600
+Wire Wire Line
+	3400 6700 3500 6700
+Wire Wire Line
+	3400 6800 3500 6800
+Text Label 2350 6650 2    50   ~ 0
+TX
+Text Label 2350 6750 2    50   ~ 0
+RX
+Text Label 2350 6900 2    50   ~ 0
+RESET
+Text Label 2350 7000 2    50   ~ 0
+MOSI
+Text Label 2350 7100 2    50   ~ 0
+MOSI
+Text Label 3500 6200 0    50   ~ 0
+D2
+Text Label 3500 6300 0    50   ~ 0
+D3
+Text Label 3500 6400 0    50   ~ 0
+D4
+Text Label 3500 6500 0    50   ~ 0
+D5
+Text Label 3500 6600 0    50   ~ 0
+D6
+Text Label 3500 6700 0    50   ~ 0
+D7
+Text Label 3500 6800 0    50   ~ 0
+D8
 $EndSCHEMATC

Commit message: Various corrections.
Connections:
- wire segments 79 -> 85
Changed lines of the file:
@@
 	6200 2400 6200 2250
 $Comp
-L power:GND #PWR?
+L power:GND #PWR0101
 U 1 1 5B805229
 P 5200 2550
-F 0 "#PWR?" H 5200 2300 50  0001 C CNN
+F 0 "#PWR0101" H 5200 2300 50  0001 C CNN
 F 1 "GND" H 5205 2377 50  0000 C CNN
 F 2 "" H 5200 2550 50  0001 C CNN
@@
 	5550 3100 5550 3350
 $Comp
-L power:GND #PWR?
+L power:GND #PWR0102
 U 1 1 5B806E4B
 P 5550 3850
-F 0 "#PWR?" H 5550 3600 50  0001 C CNN
+F 0 "#PWR0102" H 5550 3600 50  0001 C CNN
 F 1 "GND" H 5555 3677 50  0000 C CNN
 F 2 "" H 5550 3850 50  0001 C CNN
@@
 NoConn ~ 7100 4400
 $Comp
-L power:GND #PWR?
+L power:GND #PWR0103
 U 1 1 5B811509
 P 7700 4850
-F 0 "#PWR?" H 7700 4600 50  0001 C CNN
+F 0 "#PWR0103" H 7700 4600 50  0001 C CNN
 F 1 "GND" H 7705 4677 50  0000 C CNN
 F 2 "" H 7700 4850 50  0001 C CNN
@@
 ADDS2
 $Comp
-L power:GND #PWR?
+L power:GND #PWR0104
 U 1 1 5B8142A1
 P 3650 2450
-F 0 "#PWR?" H 3650 2200 50  0001 C CNN
+F 0 "#PWR0104" H 3650 2200 50  0001 C CNN
 F 1 "GND" H 3655 2277 50  0000 C CNN
 F 2 "" H 3650 2450 50  0001 C CNN
@@
 	4650 4450 4650 4300
 $Comp
-L power:GND #PWR?
+L power:GND #PWR0105
 U 1 1 5B81A59B
 P 3900 4550
-F 0 "#PWR?" H 3900 4300 50  0001 C CNN
+F 0 "#PWR0105" H 3900 4300 50  0001 C CNN
 F 1 "GND" H 3905 4377 50  0000 C CNN
 F 2 "" H 3900 4550 50  0001 C CNN
@@
 	3900 4450 4650 4450
 $Comp
-L power:PWR_FLAG #FLG?
+L power:PWR_FLAG #FLG0101
 U 1 1 5B81BD18
 P 8850 1200
-F 0 "#FLG?" H 8850 1275 50  0001 C CNN
+F 0 "#FLG0101" H 8850 1275 50  0001 C CNN
 F 1 "PWR_FLAG" H 8850 1374 50  0000 C CNN
 F 2 "" H 8850 1200 50  0001 C CNN
@@
 MOSI
 Text Label 2350 7100 2    50   ~ 0
-MOSI
+MISO
 Text Label 3500 6200 0    50   ~ 0
 D2
@@
 Text Label 3500 6800 0    50   ~ 0
 D8
+Wire Wire Line
+	3550 4100 3900 4100
+Wire Wire Line
+	3900 4100 3900 4450
+Wire Wire Line
+	5050 4100 5150 4100
+Wire Wire Line
+	5150 4100 5150 4450
+Wire Wire Line
+	5150 4450 4650 4450
+Connection ~ 4650 4450
+$Comp
+L power:PWR_FLAG #FLG0102
+U 1 1 5B841381
+P 8050 4800
+F 0 "#FLG0102" H 8050 4875 50  0001 C CNN
+F 1 "PWR_FLAG" V 8050 4928 50  0000 L CNN
+F 2 "" H 8050 4800 50  0001 C CNN
+F 3 "~" H 8050 4800 50  0001 C CNN
+	1    8050 4800
+	0    1    1    0
+$EndComp
+Wire Wire Line
+	8050 4800 7800 4800
+Connection ~ 7800 4800
 $EndSCHEMATC

Commit message: Added informational graphics.
Other:
- note added: "Atmega328P-PU with oscillator and battery"
- note added: "Clock/Calendar"
- note added: "Connectors sheet"
- note added: "EEPROM"
- moved on the sheet: U1, U3

Commit message: Created schematic for prototyping area.
Connections:
- wire segments 85 -> 87
Other:
- note added: "Prototyping area"
Changed lines of the file:
@@
 EESchema Schematic File Version 4
+LIBS:BACEE-cache
 EELAYER 26 0
 EELAYER END
 $Descr A4 11693 8268
 encoding utf-8
-Sheet 1 2
+Sheet 1 3
 Title "BACEE: Battery powered Arduino clone with Extended EEPROM"
 Date "2018-08-20"
@@
 Text Notes 3150 4600 2    50   ~ 0
 Connectors sheet
+$Sheet
+S 3550 6550 900  850
+U 5B8601B5
+F0 "prototyping_area" 50
+F1 "prototyping_area.sch" 50
+F2 "GND" I L 3550 6750 50
+F3 "5V" I L 3550 7050 50
+$EndSheet
+Text Label 3450 7050 2    50   ~ 0
+Vcc
+$Comp
+L power:GND #PWR0106
+U 1 1 5B867438
+P 3450 6750
+F 0 "#PWR0106" H 3450 6500 50  0001 C CNN
+F 1 "GND" H 3455 6577 50  0000 C CNN
+F 2 "" H 3450 6750 50  0001 C CNN
+F 3 "" H 3450 6750 50  0001 C CNN
+	1    3450 6750
+	0    1    1    0
+$EndComp
+Wire Wire Line
+	3550 6750 3450 6750
+Wire Wire Line
+	3550 7050 3450 7050
+Wire Notes Line
+	5300 6450 2500 6450
+Wire Notes Line
+	2500 6450 2500 7500
+Wire Notes Line
+	2500 7500 5300 7500
+Wire Notes Line
+	5300 7500 5300 6450
+Text Notes 3150 6400 2    50   ~ 0
+Prototyping area
 $EndSCHEMATC
