File: BACEE.sch (KiCad schematic (older format))
At the start: 13 parts, among them U1 24LC1025, U2 DS1337S+, U3 24LC1025, U4 ATMEGA328P-AU, Y1 Crystal32768KHz, Y2 Crystal 16MHz

Commit message: Adjusted designators, units etc as per Larry's feedback.
Parts:
- removed C3: 10uF, Capacitor_SMD:C_0805_2012Metric_Pad1.15x1.40mm_HandSolder, symbol Device:CP1
- added C3: 10 uF, Capacitor_SMD:C_0805_2012Metric_Pad1.15x1.40mm_HandSolder, symbol Device:CP
- C1, C2: value 22pF -> 22 pF
- R1: value 330Ohm -> 330 Ω
- R2: value 10kOhm -> 10 kΩ
- Y1: value Crystal32768KHz -> Crystal 32768 kHz
Other:
- note added: "N1 - Clock/Calendar"
- note added: "N2 - Atmega328P-PU with oscillator and battery"
- note added: "N3 - EEPROM"
- note added: "N4 - Connectors sheet"
- note added: "N5 - Prototyping area"
- note removed: "Atmega328P-PU with oscillator and battery"
- note removed: "Clock/Calendar"
- note removed: "Connectors sheet"
- note removed: "EEPROM"
- note removed: "Prototyping area"
Changed lines of the file:
@@
 P 6150 1950
 F 0 "C1" V 5898 1950 50  0000 C CNN
-F 1 "22pF" V 5989 1950 50  0000 C CNN
+F 1 "22 pF" V 5989 1950 50  0000 C CNN
 F 2 "Capacitor_SMD:C_0805_2012Metric_Pad1.15x1.40mm_HandSolder" H 6188 1800 50  0001 C CNN
 F 3 "~" H 6150 1950 50  0001 C CNN
@@
 P 6150 2500
 F 0 "C2" V 5898 2500 50  0000 C CNN
-F 1 "22pF" V 5989 2500 50  0000 C CNN
+F 1 "22 pF" V 5989 2500 50  0000 C CNN
 F 2 "Capacitor_SMD:C_0805_2012Metric_Pad1.15x1.40mm_HandSolder" H 6188 2350 50  0001 C CNN
 F 3 "~" H 6150 2500 50  0001 C CNN
@@
 $EndComp
 $Comp
-L Device:CP1 C3
-U 1 1 5B7FD83B
-P 9450 2650
-F 0 "C3" H 9565 2696 50  0000 L CNN
-F 1 "10uF" H 9565 2605 50  0000 L CNN
-F 2 "Capacitor_SMD:C_0805_2012Metric_Pad1.15x1.40mm_HandSolder" H 9450 2650 50  0001 C CNN
-F 3 "~" H 9450 2650 50  0001 C CNN
-	1    9450 2650
-	1    0    0    -1
-$EndComp
-$Comp
 L Device:R R1
 U 1 1 5B7FD90B
 P 6100 3600
 F 0 "R1" H 6030 3554 50  0000 R CNN
-F 1 "330Ohm" H 6030 3645 50  0000 R CNN
+F 1 "330 Ω" H 6030 3645 50  0000 R CNN
 F 2 "Resistor_SMD:R_0805_2012Metric_Pad1.15x1.40mm_HandSolder" V 6030 3600 50  0001 C CNN
 F 3 "~" H 6100 3600 50  0001 C CNN
@@
 P 6900 4150
 F 0 "R2" H 6970 4196 50  0000 L CNN
-F 1 "10kOhm" H 6970 4105 50  0000 L CNN
+F 1 "10 kΩ" H 6970 4105 50  0000 L CNN
 F 2 "Resistor_SMD:R_0805_2012Metric_Pad1.15x1.40mm_HandSolder" V 6830 4150 50  0001 C CNN
 F 3 "~" H 6900 4150 50  0001 C CNN
@@
 P 2700 1650
 F 0 "Y1" V 2746 1519 50  0000 R CNN
-F 1 "Crystal32768KHz" V 2655 1519 50  0000 R CNN
+F 1 "Crystal 32768 kHz" V 2655 1519 50  0000 R CNN
 F 2 "Crystal:Crystal_SMD_MicroCrystal_CC7V-T1A-2Pin_3.2x1.5mm_HandSoldering" H 2700 1650 50  0001 C CNN
 F 3 "~" H 2700 1650 50  0001 C CNN
@@
 	10750 5200 10750 950
 Text Notes 7150 900  2    50   ~ 0
-Atmega328P-PU with oscillator and battery
+N2 - Atmega328P-PU with oscillator and battery
 Wire Notes Line
 	2500 950  2500 2800
@@
 Wire Notes Line
 	5300 3000 2500 3000
-Text Notes 3100 900  2    50   ~ 0
-Clock/Calendar
-Text Notes 2800 2950 2    50   ~ 0
-EEPROM
+Text Notes 3325 900  2    50   ~ 0
+N1 - Clock/Calendar
+Text Notes 3025 2950 2    50   ~ 0
+N3 - EEPROM
 Wire Notes Line
 	2500 4650 2500 6200
@@
 Wire Notes Line
 	5300 4650 2500 4650
-Text Notes 3150 4600 2    50   ~ 0
-Connectors sheet
+Text Notes 3375 4625 2    50   ~ 0
+N4 - Connectors sheet
 $Sheet
 S 3550 6550 900  850
@@
 Wire Notes Line
 	5300 7500 5300 6450
-Text Notes 3150 6400 2    50   ~ 0
-Prototyping area
+Text Notes 3350 6425 2    50   ~ 0
+N5 - Prototyping area
+$Comp
+L Device:CP C3
+U 1 1 5BA01A54
+P 9450 2650
+F 0 "C3" H 9568 2696 50  0000 L CNN
+F 1 "10 uF" H 9568 2605 50  0000 L CNN
+F 2 "Capacitor_SMD:C_0805_2012Metric_Pad1.15x1.40mm_HandSolder" H 9488 2500 50  0001 C CNN
+F 3 "~" H 9450 2650 50  0001 C CNN
+	1    9450 2650
+	1    0    0    -1
+$EndComp
 $EndSCHEMATC
